File: ILI9341_ESP32_GBC.kicad_sch (KiCad schematic)
At the start: 83 parts, among them J1 USB_C_Receptacle_USB2.0_16P, J2 Conn_01x05_Pin, SW1 TM-2023, SW6 K3-1290S-J1, SW7 SW_Push, SW8 SW_Push, U2 XM5062S, U4 BQ25171QWDRCRQ1, U7 ESP32-S3-WROOM-1-N16R8, U8 MAX98357AETE+T, U9 TPS61028DRCR

Commit message: Upload order version 1.3
Parts:
- removed SW6: K3-1290S-J1, easyeda2kicad:SW-SMD_K3-1290S-J1, symbol easyeda2kicad:K3-1290S-J1
- added SW13: MSK12CO2-SZ, easyeda2kicad:SW-TH_MSK12C02, symbol easyeda2kicad:MSK12CO2-SZ
- J2: now fitted; now in the parts list
- L3: value 2.2µ -> 10µ; LCSC C3002559 -> C39846645
Connections:
- net BAT+: now also SW13.2
- net GND: now also SW13.4
- net V_BATT: now also SW13.1
Other:
- company: (none) -> theBrutzler
- title: (none) -> GBCRetrofitBoard
Changed lines of the file:
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@@
 	(generator_version "8.0")
 	(paper "A4")
+	(title_block
+		(title "GBCRetrofitBoard")
+		(date "2025-01-03")
+		(rev "V1.3")
+		(company "theBrutzler")
+	)
 	(junction
 		(at 219.075 32.385)
@@
 	)
 	(junction
+		(at 25.4 105.41)
+		(diameter 0)
+		(color 0 0 0 0)
+	)
+	(junction
 		(at 212.725 95.25)
 		(diameter 0)
@@
 	)
 	(junction
+		(at 50.8 105.41)
+		(diameter 0)
+		(color 0 0 0 0)
+	)
+	(junction
 		(at 68.58 73.66)
 		(diameter 0)
@@
 	(wire
 		(pts
+			(xy 25.4 102.87) (xy 25.4 105.41)
+		)
+		(stroke
+			(width 0)
+			(type default)
+		)
+	)
+	(wire
+		(pts
 			(xy 219.075 34.925) (xy 231.14 34.925)
 		)
@@
 	(wire
 		(pts
-			(xy 38.1 91.44) (xy 38.1 95.25)
+			(xy 40.64 91.44) (xy 40.64 95.25)
 		)
 		(stroke
@@
 	(wire
 		(pts
+			(xy 50.8 102.87) (xy 50.8 105.41)
+		)
+		(stroke
+			(width 0)
+			(type default)
+		)
+	)
+	(wire
+		(pts
 			(xy 255.905 74.93) (xy 258.445 74.93)
 		)
@@
 	(wire
 		(pts
-			(xy 38.1 91.44) (xy 57.785 91.44)
+			(xy 40.64 91.44) (xy 57.785 91.44)
 		)
 		(stroke
@@
 	(wire
 		(pts
+			(xy 25.4 106.68) (xy 25.4 105.41)
+		)
+		(stroke
+			(width 0)
+			(type default)
+		)
+	)
+	(wire
+		(pts
 			(xy 143.51 144.145) (xy 127 144.145)
 		)
@@
 	(wire
 		(pts
+			(xy 50.8 106.68) (xy 50.8 105.41)
+		)
+		(stroke
+			(width 0)
+			(type default)
+		)
+	)
+	(wire
+		(pts
 			(xy 258.445 87.63) (xy 256.54 87.63)
 		)
@@
 	(text "#define RG_GAMEPAD_ADC1_MAP {\\\n    {RG_KEY_UP,    ADC1_CHANNEL_6, ADC_ATTEN_DB_11, 3072, 4096},\\\n    {RG_KEY_DOWN,  ADC1_CHANNEL_6, ADC_ATTEN_DB_11, 1024, 3072},\\\n    {RG_KEY_LEFT,  ADC1_CHANNEL_5, ADC_ATTEN_DB_11, 3072, 4096},\\\n    {RG_KEY_RIGHT, ADC1_CHANNEL_5, ADC_ATTEN_DB_11, 1024, 3072},\\\n}\n#define RG_GAMEPAD_GPIO_MAP {\\\n    {RG_KEY_SELECT, GPIO_NUM_16, GPIO_PULLUP_ONLY, 0},\\\n    {RG_KEY_START,  GPIO_NUM_17, GPIO_PULLUP_ONLY, 0},\\\n    {RG_KEY_MENU,   GPIO_NUM_18, GPIO_PULLUP_ONLY, 0},\\\n    {RG_KEY_OPTION, GPIO_NUM_0,  GPIO_FLOATING,    0},\\\n    {RG_KEY_A,      GPIO_NUM_15, GPIO_PULLUP_ONLY, 0},\\\n    {RG_KEY_B,      GPIO_NUM_5,  GPIO_PULLUP_ONLY, 0},\\\n}\n\n// Battery\n#define RG_BATTERY_DRIVER           1\n#define RG_BATTERY_ADC_CHANNEL      ADC1_CHANNEL_3\n#define RG_BATTERY_CALC_PERCENT(raw) (((raw) * 2.f - 3500.f) / (4200.f - 3500.f) * 100.f)\n#define RG_BATTERY_CALC_VOLTAGE(raw) ((raw) * 2.f * 0.001f)\n\n// Status LED\n#define RG_GPIO_LED                 GPIO_NUM_38\n\n// SPI Display (back up working)\n#define RG_GPIO_LCD_MISO            GPIO_NUM_NC\n#define RG_GPIO_LCD_MOSI            GPIO_NUM_12\n#define RG_GPIO_LCD_CLK             GPIO_NUM_48\n#define RG_GPIO_LCD_CS              GPIO_NUM_NC\n#define RG_GPIO_LCD_DC              GPIO_NUM_47\n#define RG_GPIO_LCD_BCKL            GPIO_NUM_39\n#define RG_GPIO_LCD_RST             GPIO_NUM_3\n\n#define RG_GPIO_SDSPI_MISO          GPIO_NUM_9\n#define RG_GPIO_SDSPI_MOSI          GPIO_NUM_11\n#define RG_GPIO_SDSPI_CLK           GPIO_NUM_13\n#define RG_GPIO_SDSPI_CS            GPIO_NUM_10\n\n// External I2S DAC\n#define RG_GPIO_SND_I2S_BCK         41\n#define RG_GPIO_SND_I2S_WS          42\n#define RG_GPIO_SND_I2S_DATA        40\n// #define RG_GPIO_SND_AMP_ENABLE      18"
 		(exclude_from_sim no)
-		(at -26.035 151.765 0)
+		(at 12.065 162.56 0)
 		(effects
 			(font
-				(size 1.27 1.27)
+				(size 1.016 1.016)
 			)
 			(justify left)
@@
 	)
 	(label "BAT+"
-		(at 38.1 91.44 0)
+		(at 40.64 91.44 0)
 		(fields_autoplaced yes)
 		(effects
@@
 		(unit 1)
 		(exclude_from_sim no)
-		(in_bom no)
+		(in_bom yes)
 		(on_board yes)
-		(dnp yes)
+		(dnp no)
 		(property "Reference" "J2"
 			(at 259.08 33.02 0)
@@
 	)
 	(symbol
+		(lib_id "easyeda2kicad:MSK12CO2-SZ")
+		(at 40.64 102.87 0)
+		(unit 1)
+		(exclude_from_sim no)
+		(in_bom yes)
+		(on_board yes)
+		(dnp no)
+		(fields_autoplaced yes)
+		(property "Reference" "SW13"
+			(at 38.1 109.855 0)
+			(effects
+				(font
+					(size 1.27 1.27)
+				)
+			)
+		)
+		(property "Value" "MSK12CO2-SZ"
+			(at 38.1 112.395 0)
+			(effects
+				(font
+					(size 1.27 1.27)
+				)
+			)
+		)
+		(property "Footprint" "easyeda2kicad:SW-TH_MSK12C02"
+			(at 40.64 113.03 0)
+			(effects
+				(font
+					(size 1.27 1.27)
+				)
+				(hide yes)
+			)
+		)
+		(property "Datasheet" ""
+			(at 40.64 102.87 0)
+			(effects
+				(font
+					(size 1.27 1.27)
+				)
+				(hide yes)
+			)
+		)
+		(property "Description" ""
+			(at 40.64 102.87 0)
+			(effects
+				(font
+					(size 1.27 1.27)
+				)
+				(hide yes)
+			)
+		)
+		(property "LCSC" "C2681568"
+			(at 40.64 115.57 0)
+			(effects
+				(font
+					(size 1.27 1.27)
+				)
+				(hide yes)
+			)
+		)
+		(pin "1"
+		)
+		(pin "3"
+		)
+		(pin "2"
+		)
+		(pin "4"
+		)
+		(pin "4"
+		)
+		(pin "4"
+		)
+		(pin "4"
+		)
+		(instances
+			(project ""
+				(path "/ff5a7903-456b-49e1-a9c0-cc21ca8443ce"
+					(reference "SW13")
+					(unit 1)
+				)
+			)
+		)
+	)
+	(symbol
 		(lib_id "power:GND")
 		(at 95.885 27.305 0)
@@
 	)
 	(symbol
-		(lib_id "easyeda2kicad:K3-1290S-J1")
-		(at 38.1 102.87 0)
+		(lib_id "power:GND")
+		(at 142.24 27.305 0)
 		(unit 1)
 		(exclude_from_sim no)
@@
 		(dnp no)
 		(fields_autoplaced yes)
-		(property "Reference" "SW6"
-			(at 46.355 100.7099 0)
-			(effects
-				(font
-					(size 1.27 1.27)
-				)
-				(justify left)
-			)
-		)
-		(property "Value" "K3-1290S-J1"
-			(at 46.355 103.2499 0)
-			(effects
-				(font
-					(size 1.27 1.27)
-				)
-				(justify left)
-			)
-		)
-		(property "Footprint" "easyeda2kicad:SW-SMD_K3-1290S-J1"
-			(at 38.1 102.87 0)
-			(effects
-				(font
-					(size 1.27 1.27)
-				)
-				(hide yes)
-			)
-		)
-		(property "Datasheet" "https://lcsc.com/product-detail/Toggle-Switches_Korean-Hroparts-Elec-K3-1290S-J1_C223846.html"
-			(at 38.1 105.41 0)
+		(property "Reference" "#PWR016"
+			(at 142.24 33.655 0)
 			(effects
 				(font
@@
 			)
 		)
-		(property "Description" ""
-			(at 38.1 102.87 0)
+		(property "Value" "GND"
+			(at 142.24 31.75 0)
 			(effects
 				(font
 					(size 1.27 1.27)
 				)
-				(hide yes)
 			)
 		)
-		(property "LCSC Part" "C223846"
-			(at 38.1 107.95 0)
+		(property "Footprint" ""
+			(at 142.24 27.305 0)
 			(effects
 				(font
@@
 			)
 		)
-		(property "LCSC" "C223846"
-			(at 38.1 102.87 0)
+		(property "Datasheet" ""
+			(at 142.24 27.305 0)
 			(effects
 				(font
@@
 			)
 		)
-		(property "SOURCED" "ok"
-			(at 38.1 102.87 0)
+		(property "Description" "Power symbol creates a global label with name \"GND\" , ground"
+			(at 142.24 27.305 0)
 			(effects
 				(font
@@
 			)
 		)
-		(pin "2"
-		)
-		(pin "3"
-		)
 		(pin "1"
 		)
 		(instances
-			(project ""
+			(project "ILI9341_ESP32_GBC_V1"
 				(path "/ff5a7903-456b-49e1-a9c0-cc21ca8443ce"
-					(reference "SW6")
+					(reference "#PWR016")
 					(unit 1)
 				)
@@
 	(symbol
 		(lib_id "power:GND")
-		(at 142.24 27.305 0)
+		(at 25.4 106.68 0)
 		(unit 1)
 		(exclude_from_sim no)
@@
 		(dnp no)
 		(fields_autoplaced yes)
-		(property "Reference" "#PWR016"
-			(at 142.24 33.655 0)
+		(property "Reference" "#PWR014"
+			(at 25.4 113.03 0)
 			(effects
 				(font
@@
 		)
 		(property "Value" "GND"
-			(at 142.24 31.75 0)
+			(at 25.4 111.125 0)
 			(effects
 				(font
@@
 		)
 		(property "Footprint" ""
-			(at 142.24 27.305 0)
+			(at 25.4 106.68 0)
 			(effects
 				(font
@@
 		)
 		(property "Datasheet" ""
-			(at 142.24 27.305 0)
+			(at 25.4 106.68 0)
 			(effects
 				(font
@@
 		)
 		(property "Description" "Power symbol creates a global label with name \"GND\" , ground"
-			(at 142.24 27.305 0)
+			(at 25.4 106.68 0)
 			(effects
 				(font
@@
 		)
 		(instances
-			(project "ILI9341_ESP32_GBC_V1"
+			(project "ILI9341_ESP32_GBC"
 				(path "/ff5a7903-456b-49e1-a9c0-cc21ca8443ce"
-					(reference "#PWR016")
+					(reference "#PWR014")
 					(unit 1)
 				)
@@
 			)
 		)
-		(property "Value" "2.2µ"
+		(property "Value" "10µ"
 			(at 69.215 54.0004 90)
 			(effects
@@
 			)
 		)
-		(property "LCSC" "C3002559"
+		(property "LCSC" "C39846645"
 			(at 69.215 56.515 0)
 			(effects
@@
 					(unit 1)
 				)
+			)
+		)
+	)
+	(symbol
+		(lib_id "power:GND")
+		(at 50.8 106.68 0)
+		(unit 1)
+		(exclude_from_sim no)
+		(in_bom yes)
+		(on_board yes)
+		(dnp no)
+		(fields_autoplaced yes)
+		(property "Reference" "#PWR010"
+			(at 50.8 113.03 0)
+			(effects
+				(font
+					(size 1.27 1.27)
+				)
+				(hide yes)
+			)
+		)
+		(property "Value" "GND"
+			(at 50.8 111.125 0)
+			(effects
+				(font
+					(size 1.27 1.27)
+				)
+			)
+		)
+		(property "Footprint" ""
+			(at 50.8 106.68 0)
+			(effects
+				(font
+					(size 1.27 1.27)
+				)
+				(hide yes)
+			)
+		)
+		(property "Datasheet" ""
+			(at 50.8 106.68 0)
+			(effects
+				(font
+					(size 1.27 1.27)
+				)
+				(hide yes)
+			)
+		)
+		(property "Description" "Power symbol creates a global label with name \"GND\" , ground"
+			(at 50.8 106.68 0)
+			(effects
+				(font
+					(size 1.27 1.27)
+				)
+				(hide yes)
+			)
+		)
+		(pin "1"
+		)
+		(instances
+			(project "ILI9341_ESP32_GBC"
+				(path "/ff5a7903-456b-49e1-a9c0-cc21ca8443ce"
+					(reference "#PWR010")
+					(unit 1)
+				)
